File: Hardware/RPI5-Scan2Go-HAT/HAT/HAT.kicad_pcb (KiCad board)
At the start: 2 copper layers, 76 x 96.5 mm, 35 parts, among them J1 RPi_GPIO, J10 Conn_01x02_Socket, J12 Conn_01x02_Socket, J13 Conn_01x02_Socket, J14 Conn_01x02_Socket, J15 Jack-DC 5V, J18 Conn_01x02_Socket, J19 Conn_01x02_Socket, J2 Conn_01x04_Socket, J20 Conn_01x05_Socket, J21 Conn_01x05_Socket, J22 Conn_01x02_Socket, J23 Conn_01x04_Socket, J24 Conn_01x02_Socket, J3 Conn_01x14_Socket, J4 Conn_01x03_Socket, J5 Conn_01x03_Socket, J6 Conn_01x03_Socket, J7 Conn_01x04_Socket, J8 Conn_01x02_Socket, J9 Conn_01x02_Socket, Q1 DMG2305UX, U1 Pico

Commit message: improved layout
Parts:
- moved J4 10.0 mm to (132.3, 145.5)
- moved J5 10.0 mm to (144.5, 145.5)
- moved J6 10.0 mm to (156.4, 145.5)
- moved J7 0.95 mm to (140.6, 130.6)
- moved J18 0.89 mm to (143.2, 123.2)
- moved J23 0.53 mm to (140.6, 137.2)
- moved J20 0.46 mm to (122.8, 130.6)
- moved J2 0.22 mm to (124.1, 123.5)
- moved J21 0.08 mm to (122.9, 137.2)
Routing:
- net Net-(J20-Pin_5): track 35.8 -> 12.4 mm
- net GND: track 7.41 -> 0.44 mm
Changed lines of the file:
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@@
 	(footprint "Connector_JST:JST_EH_B3B-EH-A_1x03_P2.50mm_Vertical"
 		(layer "F.Cu")
-		(at 166.4354 145.4704)
+		(at 156.4354 145.4704)
 		(descr "JST EH series connector, B3B-EH-A (http://www.jst-mfg.com/product/pdf/eng/eEH.pdf), generated with kicad-footprint-generator")
 		(tags "connector JST EH vertical")
@@
 	(footprint "Connector_JST:JST_EH_B5B-EH-A_1x05_P2.50mm_Vertical"
 		(layer "F.Cu")
-		(at 122.8852 130.1496)
+		(at 122.8166 130.6068)
 		(descr "JST EH series connector, B5B-EH-A (http://www.jst-mfg.com/product/pdf/eng/eEH.pdf), generated with kicad-footprint-generator")
 		(tags "connector JST EH vertical")
 		(property "Reference" "J20"
-			(at 5 -2.8 360)
+			(at 5 -2.8 0)
 			(layer "F.SilkS")
 			(effects
@@
 		)
 		(property "Value" "Conn_01x05_Socket"
-			(at 5 3.4 360)
+			(at 5 3.4 0)
 			(layer "F.Fab")
 			(effects
@@
 		)
 		(fp_text user "${REFERENCE}"
-			(at 5 1.5 360)
+			(at 5 1.5 0)
 			(layer "F.Fab")
 			(effects
@@
 	(footprint "Connector_JST:JST_EH_B4B-EH-A_1x04_P2.50mm_Vertical"
 		(layer "F.Cu")
-		(at 124.3514 123.5202)
+		(at 124.1352 123.5202)
 		(descr "JST EH series connector, B4B-EH-A (http://www.jst-mfg.com/product/pdf/eng/eEH.pdf), generated with kicad-footprint-generator")
 		(tags "connector JST EH vertical")
 		(property "Reference" "J2"
-			(at 3.75 -2.8 360)
+			(at 3.7157 -2.3876 0)
 			(layer "F.SilkS")
 			(effects
@@
 		)
 		(property "Value" "Conn_01x04_Socket"
-			(at 17.5676 3.2476 360)
+			(at 17.5676 3.2476 0)
 			(layer "F.Fab")
 			(effects
@@
 		)
 		(fp_text user "${REFERENCE}"
-			(at 3.75 1.5 360)
+			(at 3.75 1.5 0)
 			(layer "F.Fab")
 			(effects
@@
 	(footprint "Connector_JST:JST_EH_B4B-EH-A_1x04_P2.50mm_Vertical"
 		(layer "F.Cu")
-		(at 140.1718 137.0076)
+		(at 140.649 137.241)
 		(descr "JST EH series connector, B4B-EH-A (http://www.jst-mfg.com/product/pdf/eng/eEH.pdf), generated with kicad-footprint-generator")
 		(tags "connector JST EH vertical")
 		(property "Reference" "J23"
-			(at 3.75 -2.8 360)
+			(at 3.75 -2.8 0)
 			(layer "F.SilkS")
 			(effects
@@
 		)
 		(property "Value" "Conn_01x04_Socket"
-			(at 3.75 3.4 360)
+			(at 3.75 3.4 0)
 			(layer "F.Fab")
 			(effects
@@
 		)
 		(fp_text user "${REFERENCE}"
-			(at 3.75 1.5 360)
+			(at 3.75 1.5 0)
 			(layer "F.Fab")
 			(effects
@@
 		(tags "connector barrel jack")
 		(property "Reference" "J15"
-			(at 0 -2.5 360)
+			(at 0 -2.5 0)
 			(layer "F.SilkS")
 			(effects
@@
 		)
 		(property "Value" "Jack-DC 5V"
-			(at 0 15.5 360)
+			(at 0 15.5 0)
 			(layer "F.Fab")
 			(effects
@@
 		)
 		(fp_text user "${REFERENCE}"
-			(at 0 7.5 360)
+			(at 0 7.5 0)
 			(layer "F.Fab")
 			(effects
@@
 	(footprint "Connector_JST:JST_EH_B3B-EH-A_1x03_P2.50mm_Vertical"
 		(layer "F.Cu")
-		(at 142.3454 145.4704)
+		(at 132.3454 145.4704)
 		(descr "JST EH series connector, B3B-EH-A (http://www.jst-mfg.com/product/pdf/eng/eEH.pdf), generated with kicad-footprint-generator")
 		(tags "connector JST EH vertical")
@@
 		(tags "capacitor handsolder")
 		(property "Reference" "C1"
-			(at 0 -1.85 270)
+			(at 0 -1.85 -90)
 			(layer "F.SilkS")
 			(effects
@@
 		)
 		(property "Value" "0.1uF"
-			(at 0 1.85 270)
+			(at 0 1.85 -90)
 			(layer "F.Fab")
 			(effects
@@
 		)
 		(fp_text user "${REFERENCE}"
-			(at 0 0 270)
+			(at 0 0 -90)
 			(layer "F.Fab")
 			(effects
@@
 		(tags "solder jumper open")
 		(property "Reference" "JP2"
-			(at 0 -1.8 360)
+			(at 0 -1.8 0)
 			(layer "F.SilkS")
 			(effects
@@
 		)
 		(property "Value" "Jumper_2_Open"
-			(at 0 1.9 360)
+			(at 0 1.9 0)
 			(layer "F.Fab")
 			(effects
@@
 		(tags "solder jumper open")
 		(property "Reference" "JP1"
-			(at 0 -1.8 360)
+			(at 0 -1.8 0)
 			(layer "F.SilkS")
 			(effects
@@
 		)
 		(property "Value" "Jumper_2_Open"
-			(at 0 1.9 360)
+			(at 0 1.9 0)
 			(layer "F.Fab")
 			(effects
@@
 	(footprint "Connector_JST:JST_EH_B4B-EH-A_1x04_P2.50mm_Vertical"
 		(layer "F.Cu")
-		(at 140.1572 131.4402)
+		(at 140.6182 130.6068)
 		(descr "JST EH series connector, B4B-EH-A (http://www.jst-mfg.com/product/pdf/eng/eEH.pdf), generated with kicad-footprint-generator")
 		(tags "connector JST EH vertical")
 		(property "Reference" "J7"
-			(at 3.75 -2.8 360)
+			(at 3.75 -2.8 0)
 			(layer "F.SilkS")
 			(effects
@@
 		)
 		(property "Value" "Conn_01x04_Socket"
-			(at 3.75 3.4 360)
+			(at 3.75 3.4 0)
 			(layer "F.Fab")
 			(effects
@@
 		)
 		(fp_text user "${REFERENCE}"
-			(at 3.75 1.5 360)
+			(at 3.75 1.5 0)
 			(layer "F.Fab")
 			(effects
@@
 	(footprint "Connector_JST:JST_EH_B2B-EH-A_1x02_P2.50mm_Vertical"
 		(layer "F.Cu")
-		(at 142.28 123.2408)
+		(at 143.1718 123.2408)
 		(descr "JST EH series connector, B2B-EH-A (http://www.jst-mfg.com/product/pdf/eng/eEH.pdf), generated with kicad-footprint-generator")
 		(tags "connector JST EH vertical")
 		(property "Reference" "J18"
-			(at 1.25 -2.8 360)
+			(at 1.25 -2.8 0)
 			(layer "F.SilkS")
 			(effects
@@
 		)
 		(property "Value" "Conn_01x02_Socket"
-			(at 1.25 3.4 360)
+			(at 1.25 3.4 0)
 			(layer "F.Fab")
 			(effects
@@
 		)
 		(fp_text user "${REFERENCE}"
-			(at 1.25 1.5 360)
+			(at 1.25 1.5 0)
 			(layer "F.Fab")
 			(effects
@@
 	(footprint "Connector_JST:JST_EH_B5B-EH-A_1x05_P2.50mm_Vertical"
 		(layer "F.Cu")
-		(at 122.889 137.3172)
+		(at 122.8852 137.241)
 		(descr "JST EH series connector, B5B-EH-A (http://www.jst-mfg.com/product/pdf/eng/eEH.pdf), generated with kicad-footprint-generator")
 		(tags "connector JST EH vertical")
 		(property "Reference" "J21"
-			(at 5 -2.8 360)
+			(at 5 -2.8 0)
 			(layer "F.SilkS")
 			(effects
@@
 		)
 		(property "Value" "Conn_01x05_Socket"
-			(at 5 3.4 360)
+			(at 5 3.4 0)
 			(layer "F.Fab")
 			(effects
@@
 		)
 		(fp_text user "${REFERENCE}"
-			(at 5 1.5 360)
+			(at 5 1.5 0)
 			(layer "F.Fab")
 			(effects
@@
 		(tags "SOT TO_SOT_SMD")
 		(property "Reference" "Q1"
-			(at 0 -2.4 270)
+			(at 0 -2.4 -90)
 			(layer "F.SilkS")
 			(effects
@@
 		)
 		(property "Value" "DMG2305UX"
-			(at 0 2.4 270)
+			(at 0 2.4 -90)
 			(layer "F.Fab")
 			(effects
@@
 		)
 		(fp_text user "${REFERENCE}"
-			(at 0 0 270)
+			(at 0 0 -90)
 			(layer "F.Fab")
 			(effects
@@
 	(footprint "Connector_JST:JST_EH_B3B-EH-A_1x03_P2.50mm_Vertical"
 		(layer "F.Cu")
-		(at 154.5374 145.4704)
+		(at 144.5374 145.4704)
 		(descr "JST EH series connector, B3B-EH-A (http://www.jst-mfg.com/product/pdf/eng/eEH.pdf), generated with kicad-footprint-generator")
 		(tags "connector JST EH vertical")
@@
 	)
 	(gr_rect
-		(start 138.7602 142.9972)
-		(end 174.7266 148.0264)
+		(start 128.7602 142.9972)
+		(end 164.7266 148.0264)
+		(stroke
+			(width 0.1)
+			(type default)
+		)
+		(fill none)
+		(layer "F.SilkS")
+	)
+	(gr_rect
+		(start 119.4816 121.1326)
+		(end 136.2202 133.5278)
+		(stroke
+			(width 0.1)
+			(type default)
+		)
+		(fill none)
+		(layer "F.SilkS")
+	)
+	(gr_rect
+		(start 137.1774 126.4666)
+		(end 151.6808 140.462)
 		(stroke
 			(width 0.1)
@@
 	)
 	(segment
-		(start 132.889 137.3172)
-		(end 139.8622 137.3172)
-		(width 0.2)
-		(layer "F.Cu")
-		(net 3)
-	)
-	(segment
-		(start 139.8622 137.3172)
-		(end 140.1718 137.0076)
+		(start 140.3622 137.3172)
+		(end 140.6718 137.0076)
 		(width 0.2)
 		(layer "F.Cu")
@@
 	)
 	(segment
-		(start 138.6418 124.393)
-		(end 132.8852 130.1496)
-		(width 0.2)
-		(layer "F.Cu")
-		(net 28)
-	)
-	(segment
-		(start 138.6418 109.1498)
-		(end 138.6418 124.393)
-		(width 0.2)
-		(layer "F.Cu")
-		(net 28)
-	)
-	(segment
